File: pcb/attiny_rc_switch_schematic.sch (EAGLE design)
At the start: 14 parts, among them U1 ATTINY85-20SU, U2 MOSFET_N-CH_IRLML2502TRPBFPG-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

Commit message: fixed signal pin, changed pads
Parts:
- removed U$8: SMD_PAD, scotts-library:SMD_PAD
- added U$7: SMD_PAD_NO_STENCIL, scotts-library:SMD_PAD_NO_STENCIL
- U$1, U$2, U$3, U$4, U$5, U$6: value SMD_PAD -> SMD_PAD_NO_STENCIL; device scotts-library:SMD_PAD -> scotts-library:SMD_PAD_NO_STENCIL
Connections:
- removed net PB0: U1.PB0
- new net PB5: U1.PB5
- net 5V: now also U$2.P$1; no longer U$1.P$1
- net GND: now also U$6.P$1, U$7.P$1; no longer U$2.P$1, U$4.P$1
- net OUT+: now also U$4.P$1; no longer U$3.P$1
- net OUT-: now also U$3.P$1; no longer U$6.P$1
- net SIG: now also U$1.P$1, U1.PB0; no longer U$8.P$1, U1.PB5
