File: pcb/attiny_rc_switch_th_schematic.sch (EAGLE design)
At the start: 14 parts, among them U1 ATTINY85-20PU, U2 MOSFET_N-CH_VN3205N3-GTO-92_M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

Commit message: fixed signal pin, changed pads
Parts:
- removed U$8: SMD_PAD, scotts-library:SMD_PAD
- added U$7: SMD_PAD_NO_STENCIL, scotts-library:SMD_PAD_NO_STENCIL
- U$1, U$2, U$3, U$4, U$5, U$6: value SMD_PAD -> SMD_PAD_NO_STENCIL; device scotts-library:SMD_PAD -> scotts-library:SMD_PAD_NO_STENCIL
Connections:
- removed net PB0: U1.PB0
- new net PB5: U1.PB5
- net GND: now also U$6.P$1; no longer U$4.P$1
- net OUT+: now also U$4.P$1; no longer U$3.P$1
- net OUT-: now also U$3.P$1; no longer U$6.P$1
- net SIG: now also U$7.P$1, U1.PB0; no longer U$8.P$1, U1.PB5
Changed lines of the file:
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@@
 </classes>
 <parts>
-<part name="U$8" library="scotts-library" library_urn="urn:adsk.wipprod:fs.file:vf.MFbvZbk2QL6CdGDPshwu4A" deviceset="SMD_PAD" device=""/>
-<part name="U$1" library="scotts-library" library_urn="urn:adsk.wipprod:fs.file:vf.MFbvZbk2QL6CdGDPshwu4A" deviceset="SMD_PAD" device=""/>
-<part name="U$2" library="scotts-library" library_urn="urn:adsk.wipprod:fs.file:vf.MFbvZbk2QL6CdGDPshwu4A" deviceset="SMD_PAD" device=""/>
-<part name="U$3" library="scotts-library" library_urn="urn:adsk.wipprod:fs.file:vf.MFbvZbk2QL6CdGDPshwu4A" deviceset="SMD_PAD" device=""/>
-<part name="U$4" library="scotts-library" library_urn="urn:adsk.wipprod:fs.file:vf.MFbvZbk2QL6CdGDPshwu4A" deviceset="SMD_PAD" device=""/>
-<part name="U$5" library="scotts-library" library_urn="urn:adsk.wipprod:fs.file:vf.MFbvZbk2QL6CdGDPshwu4A" deviceset="SMD_PAD" device=""/>
-<part name="U$6" library="scotts-library" library_urn="urn:adsk.wipprod:fs.file:vf.MFbvZbk2QL6CdGDPshwu4A" deviceset="SMD_PAD" device=""/>
 <part name="JP1" library="SparkFun-Jumpers" library_urn="urn:adsk.eagle:library:528" deviceset="JUMPER-SMT_2_NO" device="_NO-SILK" package3d_urn="urn:adsk.eagle:package:39277/1"/>
 <part name="U1" library="scotts-library" library_urn="urn:adsk.wipprod:fs.file:vf.MFbvZbk2QL6CdGDPshwu4A" deviceset="ATTINY85-20PU" device=""/>
@@
 <part name="D1" library="scotts-library" library_urn="urn:adsk.wipprod:fs.file:vf.MFbvZbk2QL6CdGDPshwu4A" deviceset="LED_3MM_OSR5JA3Z74A" device=""/>
 <part name="U2" library="scotts-library" library_urn="urn:adsk.wipprod:fs.file:vf.MFbvZbk2QL6CdGDPshwu4A" deviceset="MOSFET_N-CH_VN3205N3-G" device="TO-92_MC_MCH"/>
+<part name="U$7" library="scotts-library" library_urn="urn:adsk.wipprod:fs.file:vf.MFbvZbk2QL6CdGDPshwu4A" deviceset="SMD_PAD_NO_STENCIL" device=""/>
+<part name="U$1" library="scotts-library" library_urn="urn:adsk.wipprod:fs.file:vf.MFbvZbk2QL6CdGDPshwu4A" deviceset="SMD_PAD_NO_STENCIL" device=""/>
+<part name="U$2" library="scotts-library" library_urn="urn:adsk.wipprod:fs.file:vf.MFbvZbk2QL6CdGDPshwu4A" deviceset="SMD_PAD_NO_STENCIL" device=""/>
+<part name="U$3" library="scotts-library" library_urn="urn:adsk.wipprod:fs.file:vf.MFbvZbk2QL6CdGDPshwu4A" deviceset="SMD_PAD_NO_STENCIL" device=""/>
+<part name="U$4" library="scotts-library" library_urn="urn:adsk.wipprod:fs.file:vf.MFbvZbk2QL6CdGDPshwu4A" deviceset="SMD_PAD_NO_STENCIL" device=""/>
+<part name="U$5" library="scotts-library" library_urn="urn:adsk.wipprod:fs.file:vf.MFbvZbk2QL6CdGDPshwu4A" deviceset="SMD_PAD_NO_STENCIL" device=""/>
+<part name="U$6" library="scotts-library" library_urn="urn:adsk.wipprod:fs.file:vf.MFbvZbk2QL6CdGDPshwu4A" deviceset="SMD_PAD_NO_STENCIL" device=""/>
 </parts>
 <sheets>
@@
 <wire x1="20.32" y1="22.86" x2="20.32" y2="0" width="0.1524" layer="95"/>
 <wire x1="20.32" y1="0" x2="0" y2="0" width="0.1524" layer="95"/>
-<wire x1="78.74" y1="96.52" x2="78.74" y2="78.74" width="0.1524" layer="95"/>
-<wire x1="78.74" y1="78.74" x2="104.14" y2="78.74" width="0.1524" layer="95"/>
+<wire x1="76.2" y1="96.52" x2="76.2" y2="78.74" width="0.1524" layer="95"/>
+<wire x1="76.2" y1="78.74" x2="104.14" y2="78.74" width="0.1524" layer="95"/>
 <wire x1="104.14" y1="78.74" x2="104.14" y2="96.52" width="0.1524" layer="95"/>
-<wire x1="104.14" y1="96.52" x2="78.74" y2="96.52" width="0.1524" layer="95"/>
-<wire x1="78.74" y1="76.2" x2="104.14" y2="76.2" width="0.1524" layer="95"/>
+<wire x1="104.14" y1="96.52" x2="76.2" y2="96.52" width="0.1524" layer="95"/>
+<wire x1="76.2" y1="76.2" x2="104.14" y2="76.2" width="0.1524" layer="95"/>
 <wire x1="104.14" y1="76.2" x2="104.14" y2="63.5" width="0.1524" layer="95"/>
-<wire x1="104.14" y1="63.5" x2="78.74" y2="63.5" width="0.1524" layer="95"/>
-<wire x1="78.74" y1="63.5" x2="78.74" y2="76.2" width="0.1524" layer="95"/>
+<wire x1="104.14" y1="63.5" x2="76.2" y2="63.5" width="0.1524" layer="95"/>
+<wire x1="76.2" y1="63.5" x2="76.2" y2="76.2" width="0.1524" layer="95"/>
 <text x="2.54" y="20.32" size="2.1844" layer="95">From Drone</text>
 <text x="86.36" y="91.44" size="2.1844" layer="95">Battery</text>
@@
 </plain>
 <instances>
-<instance part="U$8" gate="G$1" x="15.24" y="15.24" smashed="yes" rot="R180"/>
-<instance part="U$1" gate="G$1" x="15.24" y="10.16" smashed="yes" rot="R180"/>
-<instance part="U$2" gate="G$1" x="15.24" y="5.08" smashed="yes" rot="R180"/>
-<instance part="U$3" gate="G$1" x="83.82" y="81.28" smashed="yes"/>
-<instance part="U$4" gate="G$1" x="83.82" y="86.36" smashed="yes"/>
-<instance part="U$5" gate="G$1" x="83.82" y="71.12" smashed="yes"/>
-<instance part="U$6" gate="G$1" x="96.52" y="66.04" smashed="yes" rot="R180"/>
 <instance part="JP1" gate="G$1" x="17.78" y="91.44" smashed="yes">
 <attribute name="NAME" x="17.78" y="94.234" size="1.778" layer="95" font="vector" align="center"/>
@@
 </instance>
 <instance part="U2" gate="A" x="144.78" y="48.26" smashed="yes" rot="MR0">
-<attribute name="NAME" x="126.6454" y="57.3786" size="2.083" layer="95" ratio="6" rot="MR0"/>
-<attribute name="VALUE" x="162.8448" y="54.8386" size="2.083" layer="96" ratio="6" rot="MR0"/>
-</instance>
+<attribute name="NAME" x="124.1054" y="57.3786" size="2.083" layer="95" ratio="6" rot="MR0"/>
+<attribute name="VALUE" x="155.2248" y="54.8386" size="2.083" layer="96" ratio="6" rot="MR0"/>
+</instance>
+<instance part="U$7" gate="G$1" x="10.16" y="15.24" smashed="yes"/>
+<instance part="U$1" gate="G$1" x="10.16" y="10.16" smashed="yes"/>
+<instance part="U$2" gate="G$1" x="10.16" y="5.08" smashed="yes"/>
+<instance part="U$3" gate="G$1" x="86.36" y="66.04" smashed="yes" rot="R180"/>
+<instance part="U$4" gate="G$1" x="86.36" y="71.12" smashed="yes" rot="R180"/>
+<instance part="U$5" gate="G$1" x="86.36" y="81.28" smashed="yes" rot="R180"/>
+<instance part="U$6" gate="G$1" x="86.36" y="86.36" smashed="yes" rot="R180"/>
 </instances>
 <busses>
@@
 </segment>
 <segment>
-<wire x1="88.9" y1="86.36" x2="91.44" y2="86.36" width="0.1524" layer="91"/>
-<pinref part="U$4" gate="G$1" pin="P$1"/>
 <label x="91.44" y="86.36" size="1.27" layer="95" xref="yes"/>
+<wire x1="91.44" y1="86.36" x2="86.36" y2="86.36" width="0.1524" layer="91"/>
+<pinref part="U$6" gate="G$1" pin="P$1"/>
 </segment>
 <segment>
@@
 </segment>
 </net>
-<net name="PB0" class="0">
+<net name="PB1" class="0">
+<segment>
+<pinref part="U1" gate="A" pin="PB1"/>
+<wire x1="5.08" y1="64.77" x2="2.54" y2="64.77" width="0.1524" layer="91"/>
+<label x="2.54" y="66.04" size="1.27" layer="95" rot="R180" xref="yes"/>
+</segment>
+</net>
+<net name="SIG" class="0">
+<segment>
+<wire x1="10.16" y1="15.24" x2="7.62" y2="15.24" width="0.1524" layer="91"/>
+<label x="7.62" y="15.24" size="1.27" layer="95" rot="R180" xref="yes"/>
+<pinref part="U$7" gate="G$1" pin="P$1"/>
+</segment>
 <segment>
 <pinref part="U1" gate="A" pin="PB0"/>
@@
 </segment>
 </net>
-<net name="PB1" class="0">
-<segment>
-<pinref part="U1" gate="A" pin="PB1"/>
-<wire x1="5.08" y1="64.77" x2="2.54" y2="64.77" width="0.1524" layer="91"/>
-<label x="2.54" y="66.04" size="1.27" layer="95" rot="R180" xref="yes"/>
-</segment>
-</net>
-<net name="SIG" class="0">
-<segment>
-<wire x1="10.16" y1="15.24" x2="7.62" y2="15.24" width="0.1524" layer="91"/>
-<label x="7.62" y="15.24" size="1.27" layer="95" rot="R180" xref="yes"/>
-<pinref part="U$8" gate="G$1" pin="P$1"/>
-</segment>
-<segment>
-<pinref part="U1" gate="A" pin="PB5"/>
-<wire x1="5.08" y1="54.61" x2="2.54" y2="54.61" width="0.1524" layer="91"/>
-<label x="2.54" y="55.88" size="1.27" layer="95" rot="R180" xref="yes"/>
-</segment>
-</net>
 <net name="OUT-" class="0">
 <segment>
-<wire x1="101.6" y1="48.26" x2="88.9" y2="48.26" width="0.1524" layer="91"/>
-<wire x1="88.9" y1="48.26" x2="88.9" y2="66.04" width="0.1524" layer="91"/>
-<wire x1="88.9" y1="66.04" x2="91.44" y2="66.04" width="0.1524" layer="91"/>
-<pinref part="U$6" gate="G$1" pin="P$1"/>
+<wire x1="101.6" y1="48.26" x2="91.44" y2="48.26" width="0.1524" layer="91"/>
+<wire x1="91.44" y1="48.26" x2="91.44" y2="66.04" width="0.1524" layer="91"/>
 <pinref part="U2" gate="A" pin="DRAIN"/>
+<wire x1="91.44" y1="66.04" x2="86.36" y2="66.04" width="0.1524" layer="91"/>
+<pinref part="U$3" gate="G$1" pin="P$1"/>
 </segment>
 </net>
@@
 <net name="OUT+" class="0">
 <segment>
-<wire x1="88.9" y1="81.28" x2="91.44" y2="81.28" width="0.1524" layer="91"/>
-<pinref part="U$3" gate="G$1" pin="P$1"/>
+<wire x1="91.44" y1="81.28" x2="88.9" y2="81.28" width="0.1524" layer="91"/>
 <label x="91.44" y="81.28" size="1.27" layer="95" xref="yes"/>
-<pinref part="U$5" gate="G$1" pin="P$1"/>
-<wire x1="88.9" y1="71.12" x2="91.44" y2="71.12" width="0.1524" layer="91"/>
+<wire x1="91.44" y1="71.12" x2="88.9" y2="71.12" width="0.1524" layer="91"/>
 <label x="91.44" y="71.12" size="1.27" layer="95" xref="yes"/>
 <wire x1="88.9" y1="71.12" x2="88.9" y2="81.28" width="0.1524" layer="91"/>
+<wire x1="88.9" y1="81.28" x2="86.36" y2="81.28" width="0.1524" layer="91"/>
 <junction x="88.9" y="81.28"/>
+<pinref part="U$5" gate="G$1" pin="P$1"/>
+<wire x1="88.9" y1="71.12" x2="86.36" y2="71.12" width="0.1524" layer="91"/>
 <junction x="88.9" y="71.12"/>
+<pinref part="U$4" gate="G$1" pin="P$1"/>
 </segment>
 <segment>
@@
 </segment>
 </net>
+<net name="PB5" class="0">
+<segment>
+<pinref part="U1" gate="A" pin="PB5"/>
+<wire x1="5.08" y1="54.61" x2="2.54" y2="54.61" width="0.1524" layer="91"/>
+<label x="2.54" y="55.88" size="1.27" layer="95" rot="R180" xref="yes"/>
+</segment>
+</net>
